File: hardware/stm32-trackball/stm32_dev.sch (KiCad schematic (older format))
At the start: 48 parts, among them J1 USB_C_Receptacle_USB2.0, J2 SWD, J3 UART, J4 SPARE, J5 Breakout, J6 Breakout, SW1 SIDE, SW2 SIDE, SW3 SW_Push, T1 Trackball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

Commit message: attempting to fix broken symbol
Parts:
- U4, U5, U6, U7: symbol josh-ic:AN48840B -> stm32_dev-rescue:AN48840B-josh-ic
Changed lines of the file:
@@
 	8850 2700 8400 2700
 $Comp
-L josh-ic:AN48840B U5
+L stm32_dev-rescue:AN48840B-josh-ic U5
 U 1 1 5F41B464
 P 7850 2700
@@
 	7350 1800 7250 1800
 $Comp
-L josh-ic:AN48840B U4
+L stm32_dev-rescue:AN48840B-josh-ic U4
 U 1 1 5F3F0D61
 P 7850 1900
@@
 TB_UP
 $Comp
-L josh-ic:AN48840B U6
+L stm32_dev-rescue:AN48840B-josh-ic U6
 U 1 1 5F4240DE
 P 7850 3500
@@
 $EndComp
 $Comp
-L josh-ic:AN48840B U7
+L stm32_dev-rescue:AN48840B-josh-ic U7
 U 1 1 5F42EACE
 P 7850 4250

Commit message: move symbol to updated kicad lib
Parts:
- U4, U5, U6, U7: symbol stm32_dev-rescue:AN48840B-josh-ic -> josh-ic:AN48840B
Changed lines of the file:
@@
 	8850 2700 8400 2700
 $Comp
-L stm32_dev-rescue:AN48840B-josh-ic U5
+L josh-ic:AN48840B U5
 U 1 1 5F41B464
 P 7850 2700
@@
 	7350 1800 7250 1800
 $Comp
-L stm32_dev-rescue:AN48840B-josh-ic U4
+L josh-ic:AN48840B U4
 U 1 1 5F3F0D61
 P 7850 1900
@@
 TB_UP
 $Comp
-L stm32_dev-rescue:AN48840B-josh-ic U6
+L josh-ic:AN48840B U6
 U 1 1 5F4240DE
 P 7850 3500
@@
 $EndComp
 $Comp
-L stm32_dev-rescue:AN48840B-josh-ic U7
+L josh-ic:AN48840B U7
 U 1 1 5F42EACE
 P 7850 4250
