File: hardware/stm32-trackball/stm32_dev.sch (KiCad schematic (older format))
At the start: 46 parts, among them J1 USB_C_Receptacle_USB2.0, J2 SWD, J3 UART, J4 Spare, J5 Breakout, J6 Breakout, SW1 SIDE, SW2 SIDE, SW3 SW_Push, T1 Trackball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

Commit message: partial layout, trackball TODO
Parts:
- removed C4: 100n, Capacitor_SMD:C_0603_1608Metric, symbol Device:C
- added H1, H2, H3: Fuduical, Fiducial:Fiducial_1mm_Mask2mm, symbol Mechanical:MountingHole
- J4: value Spare -> SPARE
- SW1, SW2: footprint josh-buttons-switches:Panasonic_EVQPUL_EVQPUC -> josh-buttons-switches:SW_Push_KMR2
Connections:
- net SPARE_1: now also U3.3 (PF1); no longer U3.2 (PF0)
- net SPARE_2: now also U3.2 (PF0); no longer U3.3 (PF1)
- net SPARE_3: now also U3.26 (PB5); no longer U3.24 (PB3)
- net SPARE_5: now also U3.24 (PB3); no longer U3.23 (PA15), U3.26 (PB5)
- net SPARE_6: now also U3.23 (PA15)
- net USB_DM renamed USB_N
- net USB_DP renamed USB_P
Changed lines of the file:
@@
 F 0 "SW2" V 3196 7102 50  0000 R CNN
 F 1 "SIDE" V 3105 7102 50  0000 R CNN
-F 2 "josh-buttons-switches:Panasonic_EVQPUL_EVQPUC" H 3150 7350 50  0001 C CNN
+F 2 "josh-buttons-switches:SW_Push_KMR2" H 3150 7350 50  0001 C CNN
 F 3 "~" H 3150 7350 50  0001 C CNN
 F 4 "C221909" H 3150 7150 50  0001 C CNN "LCSC"
@@
 Wire Wire Line
 	5300 2000 5450 2000
-$Comp
-L Device:C C4
-U 1 1 5EFBB364
-P 5150 1800
-F 0 "C4" V 5100 1900 50  0000 C CNN
-F 1 "100n" V 5200 1950 50  0000 C CNN
-F 2 "Capacitor_SMD:C_0603_1608Metric" H 5188 1650 50  0001 C CNN
-F 3 "~" H 5150 1800 50  0001 C CNN
-	1    5150 1800
-	0    1    1    0
-$EndComp
-Wire Wire Line
-	5000 1800 4950 1800
-Wire Wire Line
-	5300 1800 5450 1800
-Wire Wire Line
-	4950 1650 4950 1800
-Connection ~ 4950 1800
-Wire Wire Line
-	4950 1800 4950 2000
 Connection ~ 4950 2000
 Wire Wire Line
@@
 L power:+3V3 #PWR0103
 U 1 1 5EFBDFDD
-P 4950 1650
-F 0 "#PWR0103" H 4950 1500 50  0001 C CNN
-F 1 "+3V3" H 4965 1823 50  0000 C CNN
-F 2 "" H 4950 1650 50  0001 C CNN
-F 3 "" H 4950 1650 50  0001 C CNN
-	1    4950 1650
-	1    0    0    -1
-$EndComp
-Wire Wire Line
-	5450 1800 5450 2000
-Connection ~ 5450 2000
+P 4950 1850
+F 0 "#PWR0103" H 4950 1700 50  0001 C CNN
+F 1 "+3V3" H 4965 2023 50  0000 C CNN
+F 2 "" H 4950 1850 50  0001 C CNN
+F 3 "" H 4950 1850 50  0001 C CNN
+	1    4950 1850
+	1    0    0    -1
+$EndComp
 Wire Wire Line
 	5450 2000 5450 2200
@@
 TB_DOWN
 Text Label 6250 3600 2    50   ~ 0
-USB_DP
+USB_P
 Text Label 6250 3500 2    50   ~ 0
-USB_DM
+USB_N
 Text Label 6250 3700 2    50   ~ 0
 SWDIO
@@
 	1650 2400 2250 2400
 Text Label 3450 2400 2    50   ~ 0
-USB_DP
+USB_P
 Text Label 3450 2200 2    50   ~ 0
-USB_DM
+USB_N
 Wire Wire Line
 	3050 2200 3450 2200
@@
 F 0 "SW1" V 2096 6702 50  0000 R CNN
 F 1 "SIDE" V 2005 6702 50  0000 R CNN
-F 2 "josh-buttons-switches:Panasonic_EVQPUL_EVQPUC" H 2050 6950 50  0001 C CNN
+F 2 "josh-buttons-switches:SW_Push_KMR2" H 2050 6950 50  0001 C CNN
 F 3 "~" H 2050 6950 50  0001 C CNN
 F 4 "C221909" H 2050 6750 50  0001 C CNN "LCSC"
@@
 Wire Wire Line
 	8050 5550 8050 5600
-$Comp
-L Connector:Conn_01x06_Male J4
-U 1 1 5F3470ED
-P 5650 7250
-F 0 "J4" H 5622 7224 50  0000 R CNN
-F 1 "Spare" H 5622 7133 50  0000 R CNN
-F 2 "Connector_PinHeader_2.54mm:PinHeader_1x06_P2.54mm_Vertical" H 5650 7250 50  0001 C CNN
-F 3 "~" H 5650 7250 50  0001 C CNN
-	1    5650 7250
-	-1   0    0    -1
-$EndComp
+Text Label 3950 3000 0    50   ~ 0
+SPARE_1
 Text Label 3950 2900 0    50   ~ 0
-SPARE_1
-Text Label 3950 3000 0    50   ~ 0
 SPARE_2
-Text Label 3950 3400 0    50   ~ 0
+Text Label 3950 3600 0    50   ~ 0
 SPARE_3
 Text Label 3950 3500 0    50   ~ 0
 SPARE_4
-Text Label 3950 3600 0    50   ~ 0
+Text Label 3950 3400 0    50   ~ 0
 SPARE_5
 Wire Wire Line
-	3950 2900 4450 2900
-Wire Wire Line
-	4450 3000 3950 3000
+	3950 3000 4450 3000
+Wire Wire Line
+	4450 2900 3950 2900
+Wire Wire Line
+	4450 3600 3950 3600
+Wire Wire Line
+	4450 3500 3950 3500
 Wire Wire Line
 	4450 3400 3950 3400
-Wire Wire Line
-	4450 3500 3950 3500
-Wire Wire Line
-	4450 3600 3950 3600
 Text Label 6250 3900 2    50   ~ 0
-SPARE_5
+SPARE_6
 Wire Wire Line
 	5750 3900 6250 3900
@@
 Text Label 4950 7450 0    50   ~ 0
 SPARE_5
-Text Label 4950 7550 0    50   ~ 0
-SPARE_6
 Wire Wire Line
 	4950 7250 5450 7250
@@
 Wire Wire Line
 	4950 7450 5450 7450
-Wire Wire Line
-	4950 7550 5450 7550
 Text Label 8850 2700 2    50   ~ 0
 TB_RIGHT
@@
 Text Notes 7450 1400 0    100  ~ 0
 Hall Effect\nSensors
+Text Label 9450 3150 0    50   ~ 0
+nTB_BUTTON
+Wire Wire Line
+	9450 3150 9950 3150
+Wire Wire Line
+	9950 3150 9950 2850
+Connection ~ 9950 3150
+$Comp
+L Device:R R11
+U 1 1 5F768972
+P 9950 2700
+F 0 "R11" H 10020 2746 50  0000 L CNN
+F 1 "10K" H 10020 2655 50  0000 L CNN
+F 2 "Resistor_SMD:R_0603_1608Metric" V 9880 2700 50  0001 C CNN
+F 3 "~" H 9950 2700 50  0001 C CNN
+	1    9950 2700
+	1    0    0    -1
+$EndComp
+Wire Wire Line
+	9950 2550 9950 2500
+$Comp
+L power:+3V3 #PWR0140
+U 1 1 5F768979
+P 9950 2500
+F 0 "#PWR0140" H 9950 2350 50  0001 C CNN
+F 1 "+3V3" H 9965 2673 50  0000 C CNN
+F 2 "" H 9950 2500 50  0001 C CNN
+F 3 "" H 9950 2500 50  0001 C CNN
+	1    9950 2500
+	1    0    0    -1
+$EndComp
+$Comp
+L Mechanical:MountingHole T1
+U 1 1 5F7C8C3A
+P 10400 3150
+F 0 "T1" H 10500 3196 50  0000 L CNN
+F 1 "Trackball" H 10500 3105 50  0000 L CNN
+F 2 "josh-keyboard:TRACKBALL" H 10400 3150 50  0001 C CNN
+F 3 "~" H 10400 3150 50  0001 C CNN
+	1    10400 3150
+	1    0    0    -1
+$EndComp
+Text Notes 9700 2150 0    100  ~ 0
+Trackball
+Wire Wire Line
+	4950 1850 4950 2000
+$Comp
+L Mechanical:MountingHole H2
+U 1 1 5F00E4A6
+P 5100 6250
+F 0 "H2" H 5200 6296 50  0000 L CNN
+F 1 "Fuduical" H 5200 6205 50  0000 L CNN
+F 2 "Fiducial:Fiducial_1mm_Mask2mm" H 5100 6250 50  0001 C CNN
+F 3 "~" H 5100 6250 50  0001 C CNN
+	1    5100 6250
+	1    0    0    -1
+$EndComp
+$Comp
+L Mechanical:MountingHole H3
+U 1 1 5F014E75
+P 5100 6450
+F 0 "H3" H 5200 6496 50  0000 L CNN
+F 1 "Fuduical" H 5200 6405 50  0000 L CNN
+F 2 "Fiducial:Fiducial_1mm_Mask2mm" H 5100 6450 50  0001 C CNN
+F 3 "~" H 5100 6450 50  0001 C CNN
+	1    5100 6450
+	1    0    0    -1
+$EndComp
+$Comp
+L Mechanical:MountingHole H1
+U 1 1 5F015095
+P 5100 6050
+F 0 "H1" H 5200 6096 50  0000 L CNN
+F 1 "Fuduical" H 5200 6005 50  0000 L CNN
+F 2 "Fiducial:Fiducial_1mm_Mask2mm" H 5100 6050 50  0001 C CNN
+F 3 "~" H 5100 6050 50  0001 C CNN
+	1    5100 6050
+	1    0    0    -1
+$EndComp
+Text Label 4950 7550 0    50   ~ 0
+SPARE_6
+Wire Wire Line
+	4950 7550 5450 7550
+$Comp
+L Connector:Conn_01x06_Male J4
+U 1 1 5F02F257
+P 5650 7250
+F 0 "J4" H 5622 7224 50  0000 R CNN
+F 1 "SPARE" H 5622 7133 50  0000 R CNN
+F 2 "Connector_PinHeader_2.54mm:PinHeader_1x06_P2.54mm_Vertical" H 5650 7250 50  0001 C CNN
+F 3 "~" H 5650 7250 50  0001 C CNN
+	1    5650 7250
+	-1   0    0    -1
+$EndComp
+Wire Wire Line
+	9950 3250 9950 3150
+$Comp
+L power:GND #PWR0141
+U 1 1 5F791A29
+P 9950 3700
+F 0 "#PWR0141" H 9950 3450 50  0001 C CNN
+F 1 "GND" H 9955 3527 50  0000 C CNN
+F 2 "" H 9950 3700 50  0001 C CNN
+F 3 "" H 9950 3700 50  0001 C CNN
+	1    9950 3700
+	1    0    0    -1
+$EndComp
+Wire Wire Line
+	9950 3650 9950 3700
 $Comp
 L Switch:SW_Push SW3
@@
 	0    -1   -1   0
 $EndComp
-Wire Wire Line
-	9950 3250 9950 3150
-Text Label 9450 3150 0    50   ~ 0
-nTB_BUTTON
-Wire Wire Line
-	9450 3150 9950 3150
-Wire Wire Line
-	9950 3150 9950 2850
-Connection ~ 9950 3150
-$Comp
-L Device:R R11
-U 1 1 5F768972
-P 9950 2700
-F 0 "R11" H 10020 2746 50  0000 L CNN
-F 1 "10K" H 10020 2655 50  0000 L CNN
-F 2 "Resistor_SMD:R_0603_1608Metric" V 9880 2700 50  0001 C CNN
-F 3 "~" H 9950 2700 50  0001 C CNN
-	1    9950 2700
-	1    0    0    -1
-$EndComp
-Wire Wire Line
-	9950 2550 9950 2500
-$Comp
-L power:+3V3 #PWR0140
-U 1 1 5F768979
-P 9950 2500
-F 0 "#PWR0140" H 9950 2350 50  0001 C CNN
-F 1 "+3V3" H 9965 2673 50  0000 C CNN
-F 2 "" H 9950 2500 50  0001 C CNN
-F 3 "" H 9950 2500 50  0001 C CNN
-	1    9950 2500
-	1    0    0    -1
-$EndComp
-Wire Wire Line
-	9950 3650 9950 3700
-$Comp
-L power:GND #PWR0141
-U 1 1 5F791A29
-P 9950 3700
-F 0 "#PWR0141" H 9950 3450 50  0001 C CNN
-F 1 "GND" H 9955 3527 50  0000 C CNN
-F 2 "" H 9950 3700 50  0001 C CNN
-F 3 "" H 9950 3700 50  0001 C CNN
-	1    9950 3700
-	1    0    0    -1
-$EndComp
-$Comp
-L Mechanical:MountingHole T1
-U 1 1 5F7C8C3A
-P 10400 3150
-F 0 "T1" H 10500 3196 50  0000 L CNN
-F 1 "Trackball" H 10500 3105 50  0000 L CNN
-F 2 "josh-keyboard:TRACKBALL" H 10400 3150 50  0001 C CNN
-F 3 "~" H 10400 3150 50  0001 C CNN
-	1    10400 3150
-	1    0    0    -1
-$EndComp
-Text Notes 9700 2150 0    100  ~ 0
-Trackball
 $EndSCHEMATC

Commit message: Flipped TB_UP and TB_RIGHT for more convenient routing on the trackball. Almost finished routing, pad-on-pad issues with the Switch and Trackball footprints prevent routing GNDs
Connections:
- net TB_RIGHT: now also J5.6 (Pin_6), J6.6 (Pin_6), U3.12 (PA6); no longer J5.5 (Pin_5), J6.5 (Pin_5), U3.11 (PA5)
- net TB_UP: now also J5.5 (Pin_5), J6.5 (Pin_5), U3.11 (PA5); no longer J5.6 (Pin_6), J6.6 (Pin_6), U3.12 (PA6)
Changed lines of the file:
@@
 TB_LEFT
 Text Label 6250 3200 2    50   ~ 0
+TB_UP
+Text Label 6250 3300 2    50   ~ 0
 TB_RIGHT
-Text Label 6250 3300 2    50   ~ 0
-TB_UP
 Text Label 6250 3400 2    50   ~ 0
 TB_DOWN
@@
 TB_LEFT
 Text Label 6000 5850 0    50   ~ 0
-TB_RIGHT
+TB_UP
 Text Label 6000 6050 0    50   ~ 0
 TB_DOWN
@@
 	6000 5950 6500 5950
 Text Label 6000 5950 0    50   ~ 0
-TB_UP
+TB_RIGHT
 $Comp
 L power:GND #PWR0112
@@
 TB_LEFT
 Text Label 7900 5850 2    50   ~ 0
-TB_RIGHT
+TB_UP
 Text Label 7900 6050 2    50   ~ 0
 TB_DOWN
@@
 	7900 5950 7400 5950
 Text Label 7900 5950 2    50   ~ 0
-TB_UP
+TB_RIGHT
 Text Notes 1950 850  0    197  ~ 0
 STM32F042 Development

Commit message: add mounting holes to schematic, improve decoupling cap placement
Parts:
- added H4, H5, H6, H7, H8, H9: M2, MountingHole:MountingHole_2.2mm_M2, symbol Mechanical:MountingHole
Other:
- note added: "Mounting Holes"
- moved on the sheet: C1, C3, F1, J1, RN1A, RN1B, U1, U2

Commit message: added extra buttons
Parts:
- added R12, R13, R14: 10K, Resistor_SMD:R_0603_1608Metric, symbol Device:R
- added SW4, SW5, SW6: KMR2, josh-buttons-switches:SW_Push_KMR2, symbol Switch:SW_Push
- SW1, SW2: value SIDE -> KMR2
Connections:
- net +3V3: now also R12.1, R13.1, R14.1
- net GND: now also SW4.1, SW5.1, SW6.1
- net SPARE_4: now also R12.2, SW4.2
- net SPARE_5: now also R13.2, SW5.2
- net SPARE_6: now also R14.2, SW6.2
Other:
- note added: "Spare Buttons"
- moved on the sheet: R11, SW3, T1

Commit message: off to fab
Parts:
- added H10: Title, josh-logos:board-title, symbol Mechanical:MountingHole
Changed lines of the file:
@@
 Wire Wire Line
 	10950 1950 10950 2000
+$Comp
+L Mechanical:MountingHole H10
+U 1 1 5F0266C3
+P 5100 5850
+F 0 "H10" H 5200 5896 50  0000 L CNN
+F 1 "Title" H 5200 5805 50  0000 L CNN
+F 2 "josh-logos:board-title" H 5100 5850 50  0001 C CNN
+F 3 "~" H 5100 5850 50  0001 C CNN
+	1    5100 5850
+	1    0    0    -1
+$EndComp
 $EndSCHEMATC
