File: hardware/stm32-trackball-2U/stm32_dev.kicad_pcb (KiCad board)
At the start: 2 copper layers, 38.5 x 19 mm, 48 parts, among them J1 USB_C_Receptacle_USB2.0, J2 USB, Q3 DTC123J, SW1 SW_Push, SW2 BIG, SW3 SW_Push, SW4 BIG, T1 Trackball, U1 AP2112K-3.3, U2 USBLC6-2SC6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

Commit message: off to fab
Other:
- board text added: "JLCJLCJLC"
Changed lines of the file:
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@@
   (general
     (thickness 1.6)
-    (drawings 9)
+    (drawings 10)
     (tracks 518)
     (zones 0)
@@
       (outputformat 1)
       (mirror false)
-      (drillshape 1)
+      (drillshape 0)
       (scaleselection 1)
-      (outputdirectory ""))
+      (outputdirectory "./gerbers"))
   )
   (net 0 "")
@@
       (effects (font (size 1 1) (thickness 0.15)) (justify mirror))
     )
-    (fp_text user 2020-07-04 (at -2.8 -1.6) (layer Bottom)
+    (fp_text user 2020-07-04 (at -2.8 -1.6) (layer B.Mask)
       (effects (font (size 1 1) (thickness 0.15)) (justify mirror))
     )
@@
     )
   )
+  (gr_text JLCJLCJLC (at 153.2 110 90) (layer B.SilkS)
+    (effects (font (size 1 1) (thickness 0.15)) (justify mirror))
+  )
   (gr_text PWR (at 168 105) (layer B.SilkS)

Commit message: Fast forward to KiCad 7 ;)
Other:
- net class Default removed
